File: Reflow.kicad_pcb (KiCad board)
At the start: 2 copper layers, 68.6 x 53.3 mm, 35 parts, among them IC1 AD8495, IC2 AD8495, J1 Screw_Terminal_01x02, J2 Screw_Terminal_01x02, J3 Screw_Terminal_01x02, J4 Screw_Terminal_01x02, J5 Screw_Terminal_01x02, J6 Screw_Terminal_01x02, P1 Power, P2 Analog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

Commit message: Added low-pass filter on outputs.
Parts:
- added C10: 1u, Capacitor_THT:C_Rect_L7.2mm_W4.5mm_P5.00mm_FKS2_FKP2_MKS2_MKP2, F.Cu at (159.9, 119.4)
- added C11: 1u, Capacitor_THT:C_Rect_L7.2mm_W4.5mm_P5.00mm_FKS2_FKP2_MKS2_MKP2, F.Cu at (165.6, 119.4)
- added C12: 100n, Capacitor_SMD:C_0805_2012Metric, F.Cu at (139.6, 109.9)
- added C13: 100n, Capacitor_SMD:C_0805_2012Metric, F.Cu at (139.6, 88.3)
- added R10: 4k7, Resistor_SMD:R_0805_2012Metric, F.Cu at (139.6, 84.5)
- added R9: 4k7, Resistor_SMD:R_0805_2012Metric, F.Cu at (139.6, 106.0)
Connections:
- IC1 pad 5: A1 -> Net-(IC1-Pad5)
- IC1 pad 6: A1 -> Net-(IC1-Pad5)
- IC2 pad 5: A2 -> Net-(IC2-Pad5)
- IC2 pad 6: A2 -> Net-(IC2-Pad5)
Routing:
- net Net-(IC1-Pad5): track 0.00 -> 3.96 mm
- net Net-(IC2-Pad5): track 0.00 -> 3.94 mm
- net A2: track 54.8 -> 52.0 mm
- net A4: track 12.9 -> 13.9 mm
- net A1: track 47.4 -> 46.6 mm
